File: Projekty/Przylacze/PrzylaczePCB/PrzylaczePCB.kicad_sch (KiCad schematic)
At the start: 38 parts, among them J1 Conn_02x04_Odd_Even, J2 Conn_02x20_Odd_Even, J3 Conn_01x06, J4 USB_B, J5 Screw_Terminal_01x06, Q1 BC557, Q2 BC547, Q3 BC557, Q4 BC547, Q5 2N3904, Q6 2N3904, Q7 BC557, Q8 BC557, SW1 SW_Push, U1 74AHC1G04, U10 LDL1117S33R, U2 74AHC1G04, U3 ATSAM4S2AA-AU, U9 DI78M05UAB

Commit message: Przyłącze - projekt PCB v0.4
Connections:
- net GND: now also J3.6 (Pin_6); no longer J3.1 (Pin_1)
- net OPTO_R1: now also U3.35 (PA1/PGMEN1); no longer U3.32 (PA2/PGMEN2)
- net OPTO_SW2: now also U3.32 (PA2/PGMEN2); no longer U3.35 (PA1/PGMEN1)
- net at U3.25 (TDI/PB4): now also J3.1 (Pin_1); no longer J3.4 (Pin_4)
- net at U3.37 (TDO/TRACESWO/PB5): now also J3.2 (Pin_2); no longer J3.5 (Pin_5)
- net at U3.38 (JTAGSEL): now also J3.3 (Pin_3); no longer J3.2 (Pin_2)
- net at U3.39 (TMS/SWDIO/PB6): now also J3.4 (Pin_4); no longer J3.6 (Pin_6)
- net at U3.40 (TCK/SWCLK/PB7): now also J3.5 (Pin_5); no longer J3.3 (Pin_3)
Changed lines of the file:
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@@
     (stroke (width 0) (type default))
   )
+  (wire (pts (xy 236.22 68.58) (xy 236.22 60.96))
+    (stroke (width 0) (type default))
+  )
   (wire (pts (xy 193.04 121.92) (xy 191.77 121.92))
     (stroke (width 0) (type default))
@@
     (stroke (width 0) (type default))
   )
+  (wire (pts (xy 223.52 73.66) (xy 241.3 73.66))
+    (stroke (width 0) (type default))
+  )
   (wire (pts (xy 53.34 73.66) (xy 57.15 73.66))
     (stroke (width 0) (type default))
@@
     (stroke (width 0) (type default))
   )
+  (wire (pts (xy 238.76 71.12) (xy 238.76 66.04))
+    (stroke (width 0) (type default))
+  )
   (wire (pts (xy 55.88 101.6) (xy 55.88 107.95))
     (stroke (width 0) (type default))
@@
     (stroke (width 0) (type default))
   )
+  (wire (pts (xy 191.77 68.58) (xy 236.22 68.58))
+    (stroke (width 0) (type default))
+  )
   (wire (pts (xy 191.77 43.18) (xy 203.2 43.18))
     (stroke (width 0) (type default))
@@
     (stroke (width 0) (type default))
   )
-  (wire (pts (xy 256.54 57.15) (xy 256.54 58.42))
+  (wire (pts (xy 233.68 58.42) (xy 257.81 58.42))
     (stroke (width 0) (type default))
   )
@@
     (stroke (width 0) (type default))
   )
+  (wire (pts (xy 191.77 71.12) (xy 238.76 71.12))
+    (stroke (width 0) (type default))
+  )
   (wire (pts (xy 53.34 30.48) (xy 55.88 30.48))
     (stroke (width 0) (type default))
@@
     (stroke (width 0) (type default))
   )
-  (wire (pts (xy 191.77 71.12) (xy 257.81 71.12))
-    (stroke (width 0) (type default))
-  )
   (wire (pts (xy 118.11 55.88) (xy 111.76 55.88))
     (stroke (width 0) (type default))
@@
     (stroke (width 0) (type default))
   )
+  (wire (pts (xy 233.68 66.04) (xy 233.68 58.42))
+    (stroke (width 0) (type default))
+  )
   (wire (pts (xy 43.18 110.49) (xy 46.99 110.49))
     (stroke (width 0) (type default))
@@
     (stroke (width 0) (type default))
   )
+  (wire (pts (xy 191.77 63.5) (xy 223.52 63.5))
+    (stroke (width 0) (type default))
+  )
   (wire (pts (xy 118.11 81.28) (xy 106.68 81.28))
     (stroke (width 0) (type default))
@@
     (stroke (width 0) (type default))
   )
+  (wire (pts (xy 254 71.12) (xy 257.81 71.12))
+    (stroke (width 0) (type default))
+  )
   (wire (pts (xy 90.17 160.02) (xy 92.71 160.02))
     (stroke (width 0) (type default))
@@
     (stroke (width 0) (type default))
   )
+  (wire (pts (xy 231.14 63.5) (xy 257.81 63.5))
+    (stroke (width 0) (type default))
+  )
   (wire (pts (xy 261.62 85.09) (xy 264.16 85.09))
     (stroke (width 0) (type default))
@@
     (stroke (width 0) (type default))
   )
+  (wire (pts (xy 238.76 66.04) (xy 257.81 66.04))
+    (stroke (width 0) (type default))
+  )
   (wire (pts (xy 24.13 101.6) (xy 25.4 101.6))
     (stroke (width 0) (type default))
@@
     (stroke (width 0) (type default))
   )
-  (wire (pts (xy 191.77 66.04) (xy 257.81 66.04))
+  (wire (pts (xy 191.77 66.04) (xy 233.68 66.04))
     (stroke (width 0) (type default))
   )
@@
     (stroke (width 0) (type default))
   )
+  (wire (pts (xy 241.3 68.58) (xy 257.81 68.58))
+    (stroke (width 0) (type default))
+  )
   (wire (pts (xy 246.38 95.25) (xy 248.92 95.25))
     (stroke (width 0) (type default))
@@
     (stroke (width 0) (type default))
   )
-  (wire (pts (xy 200.66 60.96) (xy 257.81 60.96))
-    (stroke (width 0) (type default))
-  )
   (wire (pts (xy 17.78 68.58) (xy 17.78 69.85))
     (stroke (width 0) (type default))
@@
     (stroke (width 0) (type default))
   )
+  (wire (pts (xy 223.52 63.5) (xy 223.52 73.66))
+    (stroke (width 0) (type default))
+  )
   (wire (pts (xy 251.46 25.4) (xy 252.73 25.4))
     (stroke (width 0) (type default))
@@
     (stroke (width 0) (type default))
   )
-  (wire (pts (xy 191.77 68.58) (xy 257.81 68.58))
+  (wire (pts (xy 236.22 60.96) (xy 257.81 60.96))
     (stroke (width 0) (type default))
   )
@@
     (stroke (width 0) (type default))
   )
-  (wire (pts (xy 256.54 58.42) (xy 257.81 58.42))
-    (stroke (width 0) (type default))
-  )
   (wire (pts (xy 33.02 147.32) (xy 41.91 147.32))
     (stroke (width 0) (type default))
   )
-  (wire (pts (xy 191.77 63.5) (xy 257.81 63.5))
-    (stroke (width 0) (type default))
-  )
-  (wire (pts (xy 191.77 58.42) (xy 200.66 58.42))
+  (wire (pts (xy 191.77 58.42) (xy 231.14 58.42))
     (stroke (width 0) (type default))
   )
@@
     (stroke (width 0) (type default))
   )
+  (wire (pts (xy 241.3 73.66) (xy 241.3 68.58))
+    (stroke (width 0) (type default))
+  )
   (wire (pts (xy 78.74 167.64) (xy 80.01 167.64))
     (stroke (width 0) (type default))
@@
     (stroke (width 0) (type default))
   )
-  (wire (pts (xy 200.66 58.42) (xy 200.66 60.96))
+  (wire (pts (xy 231.14 58.42) (xy 231.14 63.5))
     (stroke (width 0) (type default))
   )
@@
     (fill (type none))
   )
-  (rectangle (start 247.65 52.07) (end 278.13 73.66)
+  (rectangle (start 247.65 55.88) (end 278.13 73.66)
     (stroke (width 0.254) (type dot) (color 0 0 255 1))
     (fill (type none))
@@
     (effects (font (size 1.778 1.778) bold) (justify left bottom))
   )
-  (global_label "OPTO_R1" (shape input) (at 100.33 83.82 180) (fields_autoplaced)
+  (global_label "OPTO_R1" (shape input) (at 100.33 80.01 180) (fields_autoplaced)
     (effects (font (size 1.27 1.27)) (justify right))
-    (property "Intersheetrefs" "${INTERSHEET_REFS}" (at 89.0785 83.82 0)
+    (property "Intersheetrefs" "${INTERSHEET_REFS}" (at 89.0785 80.01 0)
       (effects (font (size 1.27 1.27)) (justify right) hide)
     )
@@
     )
   )
-  (global_label "OPTO_SW2" (shape output) (at 100.33 80.01 180) (fields_autoplaced)
+  (global_label "OPTO_SW2" (shape output) (at 100.33 83.82 180) (fields_autoplaced)
     (effects (font (size 1.27 1.27)) (justify right))
-    (property "Intersheetrefs" "${INTERSHEET_REFS}" (at 87.6876 80.01 0)
+    (property "Intersheetrefs" "${INTERSHEET_REFS}" (at 87.6876 83.82 0)
       (effects (font (size 1.27 1.27)) (justify right) hide)
     )
@@
     )
   )
-  (symbol (lib_id "power:GND") (at 256.54 57.15 180) (unit 1)
+  (symbol (lib_id "power:GND") (at 254 71.12 270) (unit 1)
     (in_bom yes) (on_board yes) (dnp no)
-    (property "Reference" "#PWR017" (at 256.54 50.8 0)
+    (property "Reference" "#PWR017" (at 247.65 71.12 0)
       (effects (font (size 1.27 1.27)) hide)
     )
-    (property "Value" "GND" (at 256.54 53.34 0)
+    (property "Value" "GND" (at 250.19 71.12 0)
       (effects (font (size 1.27 1.27)))
     )
-    (property "Footprint" "" (at 256.54 57.15 0)
+    (property "Footprint" "" (at 254 71.12 0)
       (effects (font (size 1.27 1.27)) hide)
     )
-    (property "Datasheet" "" (at 256.54 57.15 0)
+    (property "Datasheet" "" (at 254 71.12 0)
       (effects (font (size 1.27 1.27)) hide)
     )
@@
   )
   (symbol (lib_id "Connector_Generic:Conn_01x06") (at 262.89 63.5 0) (unit 1)
-    (in_bom yes) (on_board yes) (dnp no) (fields_autoplaced)
+    (in_bom yes) (on_board yes) (dnp no)
     (property "Reference" "J3" (at 265.43 63.4999 0)
       (effects (font (size 1.27 1.27)) (justify left))
