File: Projekty/Przylacze/PrzylaczePCB/PrzylaczePCB.kicad_pcb (KiCad board)
At the start: 2 copper layers, 134.6 x 126 mm, 128 parts, among them J1 Conn_02x20_Odd_Even, J2 USB_B, J3 Conn_01x06, J4 Conn_02x04_Odd_Even, J5 Screw_Terminal_01x06, M3 MountingHole_3.2mm_M3, Q1 BC547, Q10 BC557, Q11 2N3904, Q12 2N7002, Q2 BC547, Q3 BC547, Q4 BC557, Q5 2N3904, Q6 BC557, Q7 BC557, Q8 BC547, Q9 BC557, SW1 SW_Push, SW2 SW_SPDT, SW3 SW_SPDT, SW4 SW_SPDT, SW5 SW_SPDT, SW6 SW_SPDT, SW7 SW_SPDT, SW8 SW_SPDT, SW9 SW_SPDT, U1 MCP2561-E-P, U2 ATSAM4S2AA-AU, U3 MCP2515-xSO, U4 TJA1055T_3_C,518, U5 MAX3485, U6 74AHC1G04, U7 LDL1117S33R, U8 DI78M05UAB, U9 74AHC1G04, Y1 20MHz

Commit message: Przyłącze - projekt PCB v1.3
Parts:
- added G***: LOGO, LOGO, F.Cu at (51.3, 89.0)
- added G***: LOGO, LOGO, F.Cu at (129.1, 137.9)
- added G***: LOGO, LOGO, F.Cu at (59.1, 88.8)
- moved U7 30.3 mm to (130.5, 155.3)
- moved C24 21.8 mm to (125.5, 163.3)
- moved C25 16.2 mm to (133.2, 163.3)
- moved C23 11.7 mm to (118.4, 159.9)
- moved U8 11.7 mm to (116.3, 164.1)
- moved C22 11.7 mm to (118.4, 170.8)
- moved C5 3.22 mm to (131.4, 87.2)
- moved C4 3.09 mm to (128.7, 87.2)
- moved Y1 1.90 mm to (130.4, 91.4)
Connections:
- J1 pad 10: TX_MCU -> GND
- J1 pad 11: unconnected-(J1-Pin_11-Pad11) -> TX_MCU
- J1 pad 6: unconnected-(J1-Pin_6-Pad6) -> GND
- J1 pad 8: unconnected-(J1-Pin_8-Pad8) -> GND
- J1 pad 9: unconnected-(J1-Pin_9-Pad9) -> GND
- J2 pad 4: unconnected-(J2-GND-Pad4) -> GND
- J2 pad 5: unconnected-(J2-Shield-Pad5) -> GND
Routing:
- net +3.3V: track 355.7 -> 333.9 mm
- net +12V: track 122.7 -> 106.1 mm
- net +5V: track 326.2 -> 318.7 mm
- net TX_MCU: track 237.8 -> 232.2 mm
- net Net-(U3-OSC2): track 13.3 -> 18.6 mm
- net GND: track 17.0 -> 20.7 mm, vias 16 -> 14
- net Net-(Q6-C): track 6.82 -> 5.03 mm
- net Net-(Q10-C): track 6.77 -> 5.03 mm
- net ERR: track 100.8 -> 102.3 mm
- net TXD: track 176.7 -> 178.2 mm
- net Net-(C18-Pad1): track 17.5 -> 18.9 mm
- net Net-(D12-A): track 26.5 -> 25.3 mm
- net Net-(Q1-B): track 26.4 -> 25.2 mm
- net Net-(D10-A): track 27.2 -> 28.3 mm
- net Net-(D2-K): track 64.9 -> 66.0 mm
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Other:
- board text added: "HIT IT!"
- board text added: "IT'S 106 MILES TO CHICAGO, WE'VE GOT A FULL TANK OF GAS, HALF A PACK OF CIGARETTES, IT'S DARK, AND WE'RE WEARING SUNGLASSES"
- board text added: "Przyłącze stanowiskowe v1.3 Projekt kompetencyjny 2023 6EiT Grupa 7 - Sieci przemysłowe Maciej Kaczorowski, Maciej Mierzejek, Artur Poteraj, Rafał Skwirus Politechnika Łódzka WEEIA github.com/BlackHabanero/PKgr7Sieci"
