File: Projekty/Przylacze/PrzylaczePCB/EIA485.kicad_sch (KiCad schematic)
At the start: 25 parts, among them Q10 BC557, Q11 BC547, Q12 BC547, Q9 2N7002, U4 MAX3485

Commit message: Przyłącze - projekt PCB v1.1
Parts:
- D3, D5: footprint 1_WLASNA_Library:2PAD_WIRE -> Connector_PinHeader_2.54mm:PinHeader_1x02_P2.54mm_Vertical
- Q10, Q11, Q12: footprint Package_TO_SOT_THT:TO-92_Inline -> Package_TO_SOT_THT:TO-92L_HandSolder
Changed lines of the file:
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@@
         )
         (path "/45db4533-aa6e-4785-aef0-204976ca4e66/ce7112af-9253-43da-ac3f-57b598b98707"
-          (reference "R26") (unit 1)
+          (reference "R17") (unit 1)
         )
       )
@@
       (effects (font (size 1.27 1.27)) (justify left))
     )
-    (property "Footprint" "Package_TO_SOT_THT:TO-92_Inline" (at 133.35 151.765 0)
+    (property "Footprint" "Package_TO_SOT_THT:TO-92L_HandSolder" (at 133.35 151.765 0)
       (effects (font (size 1.27 1.27) italic) (justify left) hide)
     )
@@
         )
         (path "/45db4533-aa6e-4785-aef0-204976ca4e66/ce7112af-9253-43da-ac3f-57b598b98707"
-          (reference "Q12") (unit 1)
+          (reference "Q1") (unit 1)
         )
       )
@@
         )
         (path "/45db4533-aa6e-4785-aef0-204976ca4e66/ce7112af-9253-43da-ac3f-57b598b98707"
-          (reference "C5") (unit 1)
+          (reference "C26") (unit 1)
         )
       )
@@
         )
         (path "/45db4533-aa6e-4785-aef0-204976ca4e66/ce7112af-9253-43da-ac3f-57b598b98707"
-          (reference "R15") (unit 1)
+          (reference "R28") (unit 1)
         )
       )
@@
         )
         (path "/45db4533-aa6e-4785-aef0-204976ca4e66/ce7112af-9253-43da-ac3f-57b598b98707"
-          (reference "R24") (unit 1)
+          (reference "R39") (unit 1)
         )
       )
@@
         )
         (path "/45db4533-aa6e-4785-aef0-204976ca4e66/ce7112af-9253-43da-ac3f-57b598b98707"
-          (reference "R27") (unit 1)
+          (reference "R20") (unit 1)
         )
       )
@@
         )
         (path "/45db4533-aa6e-4785-aef0-204976ca4e66/ce7112af-9253-43da-ac3f-57b598b98707"
-          (reference "R23") (unit 1)
+          (reference "R19") (unit 1)
         )
       )
@@
         )
         (path "/45db4533-aa6e-4785-aef0-204976ca4e66/ce7112af-9253-43da-ac3f-57b598b98707"
-          (reference "R25") (unit 1)
+          (reference "R40") (unit 1)
         )
       )
@@
       (effects (font (size 1.27 1.27)) (justify right))
     )
-    (property "Footprint" "1_WLASNA_Library:2PAD_WIRE" (at 130.81 130.81 0)
+    (property "Footprint" "Connector_PinHeader_2.54mm:PinHeader_1x02_P2.54mm_Vertical" (at 130.81 130.81 0)
       (effects (font (size 1.27 1.27)) hide)
     )
@@
         )
         (path "/45db4533-aa6e-4785-aef0-204976ca4e66/ce7112af-9253-43da-ac3f-57b598b98707"
-          (reference "D5") (unit 1)
+          (reference "D7") (unit 1)
         )
       )
@@
       (effects (font (size 1.27 1.27)) (justify left))
     )
-    (property "Footprint" "Package_TO_SOT_THT:TO-92_Inline" (at 88.9 149.225 0)
+    (property "Footprint" "Package_TO_SOT_THT:TO-92L_HandSolder" (at 88.9 149.225 0)
       (effects (font (size 1.27 1.27) italic) (justify left) hide)
     )
@@
         )
         (path "/45db4533-aa6e-4785-aef0-204976ca4e66/ce7112af-9253-43da-ac3f-57b598b98707"
-          (reference "Q10") (unit 1)
+          (reference "Q7") (unit 1)
         )
       )
@@
         )
         (path "/45db4533-aa6e-4785-aef0-204976ca4e66/ce7112af-9253-43da-ac3f-57b598b98707"
-          (reference "R17") (unit 1)
+          (reference "R33") (unit 1)
         )
       )
@@
         )
         (path "/45db4533-aa6e-4785-aef0-204976ca4e66/ce7112af-9253-43da-ac3f-57b598b98707"
-          (reference "C4") (unit 1)
+          (reference "C20") (unit 1)
         )
       )
@@
         )
         (path "/45db4533-aa6e-4785-aef0-204976ca4e66/ce7112af-9253-43da-ac3f-57b598b98707"
-          (reference "R18") (unit 1)
+          (reference "R29") (unit 1)
         )
       )
@@
         )
         (path "/45db4533-aa6e-4785-aef0-204976ca4e66/ce7112af-9253-43da-ac3f-57b598b98707"
-          (reference "R21") (unit 1)
+          (reference "R32") (unit 1)
         )
       )
@@
         )
         (path "/45db4533-aa6e-4785-aef0-204976ca4e66/ce7112af-9253-43da-ac3f-57b598b98707"
-          (reference "R22") (unit 1)
+          (reference "R21") (unit 1)
         )
       )
@@
         )
         (path "/45db4533-aa6e-4785-aef0-204976ca4e66/ce7112af-9253-43da-ac3f-57b598b98707"
-          (reference "R16") (unit 1)
+          (reference "R30") (unit 1)
         )
       )
@@
         )
         (path "/45db4533-aa6e-4785-aef0-204976ca4e66/ce7112af-9253-43da-ac3f-57b598b98707"
-          (reference "D4") (unit 1)
+          (reference "D11") (unit 1)
         )
       )
@@
         )
         (path "/45db4533-aa6e-4785-aef0-204976ca4e66/ce7112af-9253-43da-ac3f-57b598b98707"
-          (reference "R20") (unit 1)
+          (reference "R31") (unit 1)
         )
       )
@@
       (effects (font (size 1.27 1.27)) (justify right))
     )
-    (property "Footprint" "1_WLASNA_Library:2PAD_WIRE" (at 86.36 129.54 0)
+    (property "Footprint" "Connector_PinHeader_2.54mm:PinHeader_1x02_P2.54mm_Vertical" (at 86.36 129.54 0)
       (effects (font (size 1.27 1.27)) hide)
     )
@@
         )
         (path "/45db4533-aa6e-4785-aef0-204976ca4e66/ce7112af-9253-43da-ac3f-57b598b98707"
-          (reference "D3") (unit 1)
+          (reference "D8") (unit 1)
         )
       )
@@
         )
         (path "/45db4533-aa6e-4785-aef0-204976ca4e66/ce7112af-9253-43da-ac3f-57b598b98707"
-          (reference "Q9") (unit 1)
+          (reference "Q12") (unit 1)
         )
       )
@@
       (effects (font (size 1.27 1.27)) (justify left))
     )
-    (property "Footprint" "Package_TO_SOT_THT:TO-92_Inline" (at 114.3 167.005 0)
+    (property "Footprint" "Package_TO_SOT_THT:TO-92L_HandSolder" (at 114.3 167.005 0)
       (effects (font (size 1.27 1.27) italic) (justify left) hide)
     )
@@
         )
         (path "/45db4533-aa6e-4785-aef0-204976ca4e66/ce7112af-9253-43da-ac3f-57b598b98707"
-          (reference "Q11") (unit 1)
+          (reference "Q2") (unit 1)
         )
       )
@@
         )
         (path "/45db4533-aa6e-4785-aef0-204976ca4e66/ce7112af-9253-43da-ac3f-57b598b98707"
-          (reference "U4") (unit 1)
+          (reference "U5") (unit 1)
         )
       )
@@
         )
         (path "/45db4533-aa6e-4785-aef0-204976ca4e66/ce7112af-9253-43da-ac3f-57b598b98707"
-          (reference "R19") (unit 1)
-        )
-      )
+          (reference "R18") (unit 1)
+        )
+      )

Commit message: Przyłącze - projekt PCB v1.5
Parts:
- Q10, Q11, Q12: footprint Package_TO_SOT_THT:TO-92L_HandSolder -> Package_TO_SOT_THT:TO-92L
Changed lines of the file:
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@@
       (effects (font (size 1.27 1.27)) (justify left))
     )
-    (property "Footprint" "Package_TO_SOT_THT:TO-92L_HandSolder" (at 133.35 151.765 0)
+    (property "Footprint" "Package_TO_SOT_THT:TO-92L" (at 133.35 151.765 0)
       (effects (font (size 1.27 1.27) italic) (justify left) hide)
     )
@@
       (effects (font (size 1.27 1.27)) (justify left))
     )
-    (property "Footprint" "Package_TO_SOT_THT:TO-92L_HandSolder" (at 88.9 149.225 0)
+    (property "Footprint" "Package_TO_SOT_THT:TO-92L" (at 88.9 149.225 0)
       (effects (font (size 1.27 1.27) italic) (justify left) hide)
     )
@@
       (effects (font (size 1.27 1.27)) (justify left))
     )
-    (property "Footprint" "Package_TO_SOT_THT:TO-92L_HandSolder" (at 114.3 167.005 0)
+    (property "Footprint" "Package_TO_SOT_THT:TO-92L" (at 114.3 167.005 0)
       (effects (font (size 1.27 1.27) italic) (justify left) hide)
     )
